File: PCB/motherboard.kicad_pcb (KiCad board)
At the start: 4 copper layers, 70.9 x 38 mm, 77 parts, among them J1 USB-C In, J2 USB-C Split, J3 Pogo, J4 Extra IO, J5 SWD, J6 TC2030-NL, Q1 AO3401A, Q3 AO3400A, Q4 AO3400A, SW1 Reset, U1 STM32G0B1CCU7, U2 LMV321, U3 TPD4E05U06, U4 TPD4E05U06, U5 XC6206P332MR, U6 TPS2553

Commit message: 2026/09/17: Fixed gap in guard rail
Routing:
- net GND: track 21.7 -> 25.7 mm
Changed lines of the file:
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@@
+	)
+	(segment
+		(start 96 41.8)
+		(end 96 37.8)
+		(width 0.6)
+		(layer "B.Cu")
+		(net "GND")
 	)
 	(segment

Commit message: Progress update
Parts:
- removed J4: Extra IO, GB-Header:PinHeader_1x10_P2.54mm_Vertical-Double_Sided
- J5: moved to F.Cu
- J6: value TC2030-NL -> Conn_02x05_Odd_Even
- moved C6 92.1 mm to (130.0, 65.7)
- moved C7 92.1 mm to (128.4, 63.6)
- moved C8 92.1 mm to (133.2, 65.7)
- moved R20 92.1 mm to (135.8, 63.7)
- moved R21 92.1 mm to (135.8, 62.3)
- moved U5 92.1 mm to (130.5, 63.3)
- moved R22 92.1 mm to (136.7, 62.3)
- moved U6 92.1 mm to (133.7, 63.3)
- moved C5 52.6 mm to (131.0, 49.0)
- moved R6 52.6 mm to (131.0, 50.8)
- moved R7 52.6 mm to (131.0, 49.9)
- moved R8 52.6 mm to (131.0, 51.6)
- moved R3 52.6 mm to (134.6, 53.6)
- moved R9 52.6 mm to (129.6, 52.4)
- moved D1 52.6 mm to (132.2, 53.0)
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Connections:
- net Net-(J1-CC1) renamed CC1
- net Net-(J1-CC2) renamed CC2
- J1 pad A6: USB_D+ -> USB_A_D+
- J1 pad A7: USB_D- -> USB_A_D-
- J1 pad A8: unconnected-(J1-SBU1-PadA8) -> SBU1
- J1 pad B6: USB_D+ -> USB_B_D+
- J1 pad B7: USB_D- -> USB_B_D-
- J1 pad B8: unconnected-(J1-SBU2-PadB8) -> SBU2
- J6 pad 1: +3V3 -> unconnected-(J6-Pin_1-Pad1)
- J6 pad 2: SWDIO -> unconnected-(J6-Pin_2-Pad2)
- J6 pad 3: RST -> unconnected-(J6-Pin_3-Pad3)
- J6 pad 4: BOOT0/SWCLK -> unconnected-(J6-Pin_4-Pad4)
- J6 pad 5: GND -> unconnected-(J6-Pin_5-Pad5)
- U1 pad 12: GPIO5_POGO -> unconnected-(U1-PA1-Pad12)
- U1 pad 13: GPIO4_POGO -> unconnected-(U1-PA2-Pad13)
- U1 pad 14: GPIO3_POGO -> unconnected-(U1-PA3-Pad14)
- U1 pad 40: GPIO10_EXTRA -> unconnected-(U1-PD2-Pad40)
- U1 pad 41: GPIO9_EXTRA -> unconnected-(U1-PD3-Pad41)
- U1 pad 42: GPIO8_EXTRA -> unconnected-(U1-PB3-Pad42)
- U1 pad 43: GPIO7_EXTRA -> unconnected-(U1-PB4-Pad43)
- U1 pad 44: GPIO6_EXTRA -> unconnected-(U1-PB5-Pad44)
- U1 pad 45: GPIO5_EXTRA -> GPIO5_POGO
- U1 pad 46: GPIO4_EXTRA -> GPIO4_POGO
- U1 pad 47: GPIO3_EXTRA -> GPIO3_POGO
- U1 pad 48: GPIO2_EXTRA -> unconnected-(U1-PB9-Pad48)
Routing:
- net BOOT0/SWCLK: track 71.5 -> 3.89 mm, vias 3 -> 0
- net RST_BUTTON: track 64.0 -> 1.18 mm
- net SWDIO: track 58.2 -> 0.00 mm, vias 2 -> 0
- net RST: track 60.1 -> 2.13 mm
- net +3V3: track 51.0 -> 8.88 mm, vias 11 -> 4
- net GPIO1_EXTRA: track 30.7 -> 0.00 mm, vias 1 -> 0
- net VBUS_DET: track 34.5 -> 5.36 mm, vias 2 -> 1
- net USB_D-: track 39.7 -> 24.0 mm
- net GPIO2_EXTRA: track 15.5 -> 0.00 mm
- net USB_D+: track 40.4 -> 25.7 mm
- net GPIO3_EXTRA: track 13.5 -> 0.00 mm
- net GPIO4_EXTRA: track 11.5 -> 0.00 mm
- net GND: track 25.7 -> 14.2 mm, vias 190 -> 122
- net RGB_EN: track 10.1 -> 0.00 mm
- net GPIO5_EXTRA: track 9.52 -> 0.00 mm
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- added copper zone on F.Cu, net /VREF
- removed copper zone on In2.Cu, net +3V3
- removed copper zone on In2.Cu, net +5V
- removed copper zone on In2.Cu, net VBUS
Other:
- board size 70.9 x 38 mm -> 50 x 38 mm
- board text removed: "3V3"
- board text removed: "5V"
- board text removed: "A15"
- board text removed: "B3"
- board text removed: "B4"
- board text removed: "B5"
- board text removed: "B6"
- board text removed: "B7"
- board text removed: "B8"
- board text removed: "B9"
- board text removed: "CS"
- board text removed: "D2"
- board text removed: "D3"
- board text removed: "EXTRA GPIO"
- board text removed: "GP1"
- board text removed: "GP2"
- board text removed: "GP3"
- board text removed: "GP4"
- board text removed: "GP5"
- board text removed: "Hold down button for 3 secs to enter"
- board text removed: "MIS"
- board text removed: "MOS"
- board text removed: "RESET"
- board text removed: "RGB"
- board text removed: "SCK"
- board text removed: "SCL"
- board text removed: "SDA"
- board text removed: "VIK OUT"
- board text removed: "device bootloader"
