File: PCB/motherboard.kicad_sch (KiCad schematic)
At the start: 75 parts, among them J1 USB-C In, J2 USB-C Split, J3 Pogo, J4 Extra IO, J5 SWD, J6 TC2030-NL, Q1 AO3401A, Q3 AO3400A, Q4 AO3400A, SW1 Reset, U1 STM32G0B1CCU7, U2 LMV321, U3 TPD4E05U06, U4 TPD4E05U06, U5 XC6206P332MR, U6 TPS2553

Commit message: Progress update
Parts:
- removed J4: Extra IO, GB-Header:PinHeader_1x10_P2.54mm_Vertical-Double_Sided, symbol Connector_Generic:Conn_01x10
- removed J6: TC2030-NL, GB-Header:Paw-Connect_RevB_TC2030-IDC-NL_2x03_P1.27mm_Vertical_Double-Sided, symbol Connector:Conn_ARM_SWD_TagConnect_TC2030-NL
- added J6: Conn_02x05_Odd_Even, symbol Connector_Generic:Conn_02x05_Odd_Even
Connections:
- net GPIO3_EXTRA is gone; now on net GPIO3_POGO: U1.47 (PB8)
- net GPIO4_EXTRA is gone; now on net GPIO4_POGO: U1.46 (PB7)
- net GPIO5_EXTRA is gone; now on net GPIO5_POGO: U1.45 (PB6)
- net GPIO3_POGO: no longer U1.14 (PA3)
- net GPIO4_POGO: no longer U1.13 (PA2)
- net GPIO5_POGO: no longer U1.12 (PA1)
- net USB_D+: no longer J1.A6 (D+), J1.B6 (D+)
- net USB_D-: no longer J1.A7 (D-), J1.B7 (D-)
- net CC1: now reaches J1.A5 (CC1), R11.1
- net SBU1: now reaches J1.A8 (SBU1)
- net CC2: now reaches J1.B5 (CC2), R10.1
- net SBU2: now reaches J1.B8 (SBU2)
- net GPIO10_EXTRA: no longer names the net of U1.40 (PD2)
- net GPIO2_EXTRA: no longer names the net of U1.48 (PB9)
- net GPIO6_EXTRA: no longer names the net of U1.44 (PB5)
- net GPIO7_EXTRA: no longer names the net of U1.43 (PB4)
- net GPIO8_EXTRA: no longer names the net of U1.42 (PB3)
- net GPIO9_EXTRA: no longer names the net of U1.41 (PD3)
- new net USB_A_D+: J1.A6 (D+)
- new net USB_A_D-: J1.A7 (D-)
- new net USB_B_D+: J1.B6 (D+)
- new net USB_B_D-: J1.B7 (D-)
- no-connect marks 18 -> 15
Other:
- moved on the sheet: C1, C2, C3, C4, C5, C6, C7, C8, D1, D10, D11, D12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
