File: Motherboard/Motherboard.kicad_sch (KiCad schematic)
At the start: 73 parts, among them J1 USB-C In, J2 USB-C Split, J3 Pogo, J4 Conn_ARM_JTAG_SWD_10, Q1 AO3401A, Q3 AO3400A, Q4 AO3400A, SW1 Reset, U1 STM32G0B1CCU7, U2 LMV321, U3 TPD4E05U06, U4 TPD4E05U06, U5 XC6206P332MR, U6 TPS2553D

Commit message: 2026/09/26: V0.3 motherboard update complete
Reduced size again, rerouted board and changed shape slightly. Removed one mounting hole and centred the other between the USB ports. Changed input fuse and external +5V output to TPS2553-1 latching power switch with reverse voltage/current protection. Removed AO3401 and LMV321 discrete reverse current protection at VBUS input. Reduced size of VBUS and VSPLIT ferrite bead and transistors in the Acheron reset circuit. Made Acheron reset circuit reach DFU faster.
Parts:
- removed F1, F2: 500m, GB-Device:PTC_0603_1608Metric, symbol Device:Polyfuse_Small
- removed H3: M3, GB-HolePad:MountingHole_3.2mm_M3_Pad_Via, symbol GB-Misc:MountingHole_Pad
- removed Q1: AO3401A, GB-Package:SOT-23-3, symbol Transistor_FET:AO3401A
- removed R12, R20: 100k, GB-Device:R_0402_1005Metric, symbol Device:R_Small
- removed R13, R2, R21: 200k, GB-Device:R_0402_1005Metric, symbol Device:R_Small
- removed R22: 1M, GB-Device:R_0402_1005Metric, symbol Device:R_Small
- removed U2: LMV321, GB-Package:SOT-23-5, symbol Amplifier_Operational:LMV321
- removed U5: XC6206P332MR, GB-Package:SOT-23-3, symbol Regulator_Linear:XC6206PxxxMR
- removed U6: TPS2553D, GB-Package:SOT-23-6, symbol GB-IC:TPS2553D
- added C11, C12, C5: 10u, GB-Device:C_0603_1608Metric, symbol Device:C_Small
- added C4: 100n, GB-Device:C_0402_1005Metric, symbol Device:C_Small
- added J3: SWD, Paw-Connect:Paw-Connect_RevB_TC2030-IDC-NL_2x03_P1.27mm_Vertical, symbol Connector:Conn_ARM_SWD_TagConnect_TC2030-NL
- added R17, R18, R4, R7: 100k, GB-Device:R_0402_1005Metric, symbol Device:R_Small
- added R19, R5, R9: 150k, GB-Device:R_0402_1005Metric, symbol Device:R_Small
- added U3, U5: TPS2553-1, GB-Package:WSON-6-1EP_2x2mm_P0.65mm_EP1x1.6mm, symbol GB-IC:TPS2553DR
- added U4: XC6206P332MR, GB-Package:SOT-23-3, symbol Regulator_Linear:XC6206PxxxMR
- C1: renamed from C3; Rating (none) -> 50V; Voltage 50V -> (none)
- C10: renamed from C5; Rating (none) -> 50V; Voltage 50V -> (none)
- C2: renamed from C1; Rating (none) -> 25V; Voltage 25V -> (none)
- C3: renamed from C2; Rating (none) -> 50V; Voltage 50V -> (none)
- C6, C7: Rating (none) -> 25V; Voltage 25V -> (none)
- C8: Rating (none) -> 50V; Voltage 50V -> (none)
- C9: renamed from C4; Rating (none) -> 25V; Voltage 25V -> (none)
- D2: renamed from D1; value 1N4148 -> 1N4148WT; footprint GB-Device:D_SOD-323 -> GB-Device:D_SOD-523; LCSC C2128 -> C7420320; MPN 1N4148WS -> 1N4148WT; Manufacturer Jiangsu Changjing Electronics Technology Co., Ltd. -> hongjiacheng
- FB1: renamed from FB3; value 150@100 -> 120@100; footprint GB-Device:L_0603_1608Metric -> GB-Device:L_0402_1005Metric; LCSC C404681 -> C275477; MPN MPZ1608Y151BTD25 -> MPZ1005S121ET000
- FB2: renamed from FB1; value 150@100 -> 120@100; footprint GB-Device:L_0603_1608Metric -> GB-Device:L_0402_1005Metric; LCSC C404681 -> C275477; MPN MPZ1608Y151BTD25 -> MPZ1005S121ET000
- FB3: renamed from FB2; value 150@100 -> 120@100; footprint GB-Device:L_0603_1608Metric -> GB-Device:L_0402_1005Metric; LCSC C404681 -> C275477; MPN MPZ1608Y151BTD25 -> MPZ1005S121ET000
- H1, H2: LCSC (none) -> N/A; MPN (none) -> N/A
- J1: footprint GB-Connector:USB_C_Receptacle_HRO_TYPE-C-31-M-13x -> GB-Connector:USB_C_Receptacle_Molex_2169900001; LCSC C2848620 -> C2843969; MPN TYPE-C-31-M-13C -> GT-USB-7014D; Manufacturer Korean Hroparts Elec -> G-Switch
- J2: renamed from J4; value Conn_ARM_JTAG_SWD_10 -> SWD; LCSC (none) -> N/A; MPN (none) -> FTSH-105-01-L-D-K
- J4: renamed from J3; footprint GB-Header:Connector_2x08_2.54mm_MillMax_Pogo_Target_419-10-216-00-001000-Double_Sided -> GB-Header:PinHeader_2x08_2.54mm_MillMax_PogoTarget_419-10-216-00-001000-Double_Sided; LCSC (none) -> N/A; now not fitted
- J5: renamed from J2; footprint GB-Connector:USB_C_Receptacle_HRO_TYPE-C-31-M-13x -> GB-Connector:USB_C_Receptacle_Molex_2169900001; LCSC C2848620 -> C2843969; MPN TYPE-C-31-M-13C -> GT-USB-7014D; Manufacturer Korean Hroparts Elec -> G-Switch
- JP1, TOOL1, TOOL2, TOOL3: LCSC (none) -> N/A; MPN (none) -> N/A; Manufacturer (none) -> N/A
- Q1: renamed from Q4; value AO3400A -> 2N7002W; footprint GB-Package:SOT-23-3 -> GB-Package:SOT-323_SC-70-3; LCSC C20917 -> C7420322; MPN AO3400A -> 2N7002W; Manufacturer Alpha & Omega Semiconductor Inc -> hongjiacheng
- Q2: renamed from Q3; value AO3400A -> 2N7002W; footprint GB-Package:SOT-23-3 -> GB-Package:SOT-323_SC-70-3; LCSC C20917 -> C7420322; MPN AO3400A -> 2N7002W; Manufacturer Alpha & Omega Semiconductor Inc -> hongjiacheng
- R8: value 100k -> 56k; LCSC C25741 -> C25796; MPN 0402WGF1003TCE -> 0402WGF5602TCE
- SW1: MPN (none) -> SKSNLPE010; Manufacturer (none) -> Alps Alpine
- renumbered D2 to D1, D11 to D10, D6 to D11, D14 to D12, D17 to D13, D18 to D14, D12 to D17, D13 to D18, D4 to D3, D5 to D4, D3 to D5, D7 to D6, D8 to D7, D9 to D8, D10 to D9, R18 to R1, R3 to R10, R4 to R11, R5 to R12, R6 to R13, R7 to R14, R14 to R15, R15 to R16, R10 to R2, R16 to R20, R17 to R21, R9 to R22, R11 to R3, R19 to R6, U3 to U1, U1 to U2, U4 to U6
Connections:
- net +3V3: now also J3.1 (VCC), R18.2, U4.2 (VO)
- net +5V: now also C11.2, U5.6 (OUT)
- net BOOT0/SWCLK: now also J3.4 (SWCLK), R9.2
- net I2C2_SCL: now also U2.42 (PB3); no longer U2.25 (PB13)
- net I2C2_SDA: now also U2.43 (PB4); no longer U2.26 (PB14)
- net RGB_EN: now also U2.25 (PB13), U5.3 (EN); no longer U2.28 (PA8)
- net RST: now also J3.3 (~{RESET})
- net SPLIT_SIDE: now also U2.37 (PA15); no longer U2.1 (PC13)
- net SWDIO: now also J3.2 (SWDIO)
- net VBUS: now also D5.1 (K), C12.2, C5.2, U3.6 (OUT), U4.3 (VI), U5.1 (IN)
- net VBUS_DET: now also R4.1, R5.2
- net VBUS_FERRITE: now also D1.1 (K), C4.2, R4.2, R7.2, U3.1 (IN)
- net VBUS_RAW: now also FB2.1
- net VSPLIT_RAW: now also FB3.2
- net ~{RGB_FAULT}: now also U2.24 (PB12), R18.1, U5.4 (~{FAULT}); no longer U2.27 (PB15)
- net at Q2.1 (G), R13.2: now also R17.2; no longer R8.2
- net at D2.1 (K): now also R9.1
- net CC1: no longer names the net of J1.A5 (CC1), R3.1
- net CC2: no longer names the net of J1.B5 (CC2), R2.1
- net GND renamed EP
- net EP: now also R8.2, C11.1, C12.1, C4.1, C5.1, J3.5 (GND), R17.1, R19.1, R5.1, U3.2 (GND), U3.4 (~{FAULT}), U3.7 (EP), U4.1 (GND), U5.2 (GND), U5.7 (EP); no longer R8.1
- net SPLIT_RX renamed USART1_SPLIT_RX
- net SPLIT_TX renamed USART1_SPLIT_TX
- net USART1_RX renamed USART1_MCU_RX
- net USART1_TX renamed USART1_MCU_TX
- removed net VBUS_FUSED: D1.1 (K), FB2.1
- removed net VSPLIT_FUSED: D5.1 (K), FB3.2
- new net: R19.2, U5.5 (ILIM)
- new net: R7.1, U3.3 (EN)
- new net: R8.1, U3.5 (ILIM)
- no-connect marks 27 -> 29
Other:
- note added: "Takes about 2s for boot0 to reach 1.61V."
- note added: "When R(ILIM) = 150k @ 1% ILIM (MIN) = 25230/(56^(1.016)) ~= 155mA ILIM (NOM) = 23950/(150^(0.977)) ~= 179mA ILIM (MAX) = 22980/(150^(0.94)) ~= 207mA"
- note added: "When R(ILIM) = 56k @ 1% ILIM (MIN) = 25230/(56^(1.016)) ~= 422mA ILIM (NOM) = 23950/(56^(0.977)) ~= 469mA ILIM (MAX) = 22980/(56^(0.94)) ~= 522mA"
- note added: "When VBUS = 5V5 Resistor divider = 3V3"
- note removed: "R(ILIM) = 1M || 200k @ 1% ~= 188mA"
- note removed: "Takes about 2.4s for boot0 to reach 1.61V."
- moved on the sheet: C1, C10, C2, C3, C6, C7, C8, C9, D1, D10, D11, D12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
